File: WRG_GOALCATCHER.kicad_pcb (KiCad board)
At the start: 2 copper layers, 142 x 198 mm, 136 parts, among them J1 Conn_01x03, J10 VL6180, J11 VL6180, J12 VL6180, J13 Conn_01x04, J14 Conn_01x04, J17 Conn_01x02, J2 Conn_01x02, J3 Conn_01x04_Male, J4 Conn_01x03_Pin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

Commit message: Add files via upload
Parts:
- removed H2, H3: WHEEL, PIN:Pillars-M3.2R5
- moved C4 5.90 mm to (62.7, 80.3)
- moved D5 1.22 mm to (77.8, 6.00)
- moved D8 0.23 mm to (122.7, 6.00)
- moved H8 0.20 mm to (100.0, -13.8)
Routing:
- net +3V3: track 513.0 -> 473.8 mm
- net PWM8: track 111.4 -> 100.1 mm
- net PWM0: track 97.2 -> 104.0 mm
- net GND: track 1381.0 -> 1377.1 mm
- net Net-(D5-DOUT): track 16.8 -> 19.5 mm
- net BATTERY+: track 81.7 -> 79.4 mm
- net VD: track 643.2 -> 644.9 mm
- net SCL3: track 163.4 -> 162.2 mm
- net VDC: track 141.6 -> 140.5 mm
- net SW1: track 71.7 -> 71.0 mm
- net Vdrive: track 157.4 -> 156.8 mm
- net Net-(D4-DOUT): track 19.0 -> 18.4 mm
Other:
- board text added: "+"
- board text added: "0"
- board text added: "1"
- board text added: "10"
- board text added: "11"
- board text added: "12"
- board text added: "13"
- board text added: "14"
- board text added: "15"
- board text added: "16"
- board text added: "17"
- board text added: "18"
- board text added: "19"
- board text added: "2"
- board text added: "20"
- board text added: "21"
- board text added: "22"
- board text added: "23"
- board text added: "24"
- board text added: "3"
- board text added: "3V3"
- board text added: "4"
- board text added: "5"
- board text added: "5V"
- board text added: "6"
- board text added: "7"
- board text added: "8"
- board text added: "9"
- board text added: "GND"
- board text added: "MOTO"
- board text added: "OLED"
- board text added: "RC Servo"
- board text added: "SCL"
- board text added: "SCL1"
- board text added: "SCL2"
- board text added: "SCL3"
- board text added: "SCL7"
- board text added: "SDA"
- board text added: "SDA1"
- board text added: "SDA2"
- board text added: "SDA3"
- board text added: "SDA7"
- board text added: "SPK"
- board text added: "VCC"
- board text added: "VD"
- board text added: "VDC"
- board text added: "VDD"
- board text added: "VPP"
- board text added: "Vdrive"
- board text removed: "Left Wheel"
- board text removed: "PWM0"
- board text removed: "PWM1"
- board text removed: "PWM2"
- board text removed: "PWM5"
- board text removed: "Right Wheel"
